Commit message: Add imu sensor to OREO

File: urdf/base/oreo_base.urdf.xacro (robot description, xacro)
@@ -12,5 +12,5 @@
     <joint name="dummy" type="fixed">
       <parent link="base_footprint" />
-      <child link="base_link" />
+      <child link="${link}" />
     </joint>
     <link
@@ -51,5 +51,5 @@
     <xacro:omni_wheel name="b" joint_xyz="-0.24269 0.0 0.08" joint_rpy="0 0 -3.14159265359" parent="${link}" wheel_radius="0.065" roller_radius="0.01" roller_length="0.02"/>
     <!-- laser -->
-    <xacro:sick_lms1xx parent="base_link" frame="laser" topic="scan">
+    <xacro:sick_lms1xx parent="${link}" frame="laser" topic="scan">
       <origin xyz="0.15 0 0.354" rpy="0 0 0" />
     </xacro:sick_lms1xx>

File: urdf/body/oreo_body.urdf.xacro (robot description, xacro)
@@ -8,4 +8,5 @@
   <xacro:include filename="$(find oreo_description)/urdf/sensor/camera/_d435.urdf.xacro"/>
   <xacro:include filename="$(find velodyne_description)/urdf/VLP-16.urdf.xacro"/>
+  <xacro:include filename="$(find oreo_description)/urdf/sensor/imu/imu.urdf.xacro"/>
   <xacro:macro name="oreo_body" params="link parent joint">
     <link
@@ -34,10 +35,4 @@
         </geometry>
       </visual>
-      <!-- <collision>
-        <origin xyz="0 0 0.30" rpy="0 0 0"/>
-        <geometry>
-          <cylinder length="0.60" radius="0.20"/>
-        </geometry>
-      </collision> -->
     </link>
     <joint
@@ -66,4 +61,6 @@
       <origin xyz="0.175 0 0.5825" rpy="0 0 0" />
     </xacro:sensor_d435>
+    <!-- imu -->
+    <xacro:imu name="imu" joint_xyz="0.175 0 0.5825" joint_rpy="0.0 0.0 0.0" parent="${link}" visualize="false" topic="imu"/>
     <!-- gazebo description -->
     <xacro:omni_body_gazebo link="${link}"/>
